File: kicad/AC30.kicad_sch (KiCad schematic)
At the start: 81 parts, among them IC10 555, IC11 4001, IC12 1489, IC13 4070, IC14 4053, IC15 1488, IC6 4053, IC7 4049, IC8 4013, IC9 4023, J1 Front panel harness 1, J10 MOTOR A, J11 MOTOR B, J2 Front panel harness 2, J3 Computer interface (COMP), J4 Control interface, J5 Terminal interface (TERM), J6 MIC A, J7 MIC B, J8 EAR A, J9 EAR B, Q10 2N5087, Q11 2N5087, Q5 2N5210, Q6 2N5210, Q7 2N5210, Q8 2N5210, Q9 2N5087

Commit message: Wire mod/demod and external power supply; retry routing until DRC-clean
- Transcribe docs/ac30_mod_demod.pdf onto sheet 2: modulator (IC5A/B,
  IC2A, IC4A filter) and demodulator (IC4B comparator, IC3C/D edge pulses,
  carrier detect, missing-pulse detector, R16 timer, IC1A data out, 16X
  clock out). The mod/demod interface solder pads are removed.
- Transcribe docs/ac30_PS.pdf onto new sheet 3 as an external unit (no
  footprints): line cord, S6, F1, T1, bridge D14-D17, +/-13 V, +/-7.5 V
  zener rails, 7805. IC16 GND taken as GND (drawing ties it to -13 V).
- Board gets through-hole power input pads TP1-TP6 (+5V, GND, +13V, -13V,
  +7.5V, -7.5V) with rail names on the silkscreen, plus C23-C25 +5 V
  bypass. IC4 on +/-7.5 V, IC15 on +/-13 V. J2 18 VAC pins now unused.
- Corner mounting holes H1-H4, 6.35 mm in from each edge (artwork).
- Placement weighs all nets except +5V/GND; build.sh routes the placed
  board afresh up to 4 times and keeps the first DRC-clean result.
- Board 173.0 x 121.5 mm, fully routed; ERC, DRC (all severities) and
  schematic parity clean. AC30-settings.md updated.

Co-Authored-By: Claude Opus 5.5 <noreply@anthropic.com>
Connections:
- net 18VAC_A: no longer names the net of J2.11 (Pin_11)
- net 18VAC_B: no longer names the net of J2.12 (Pin_12)
- net V_RS232+ renamed +13V
- net V_RS232- renamed -13V
- no-connect marks 32 -> 34
Other:
- sheet Mod/Demod & Power pads renamed Mod/Demod & power input
- added sheet Power supply (external) (AC30_power_supply.kicad_sch)
- moved on the sheet: C12, C13, C14, C15, C16, C17, C18, D18, D19, D20, D21, D22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

Commit message: Through-hole board: front-panel jumper pads in place of J1/J2
Both boards now wire the front panel to five rows of 0.1 in through-hole
pads with net names on the silkscreen (J1 SWITCHES, J2 LEDS, J13 MOTOR,
J14 MIC, J15 EAR) instead of the artwork's J1/J2 KK-396 headers.

The through-hole build weights board height at 60 (AC30_HEIGHT_W) so the
bottom row doesn't stretch the board; it is now 173.0 x 126.5 mm, fully
routed, ERC/DRC/parity clean. SMT board unchanged apart from symbol IDs
and the schematic note. AC30-settings.md updated.

Co-Authored-By: Claude Opus 5.5 <noreply@anthropic.com>
Parts:
- added J13: MOTOR, Connector_PinHeader_2.54mm:PinHeader_1x04_P2.54mm_Vertical, symbol Connector_Generic:Conn_01x04
- added J14: MIC, Connector_PinHeader_2.54mm:PinHeader_1x04_P2.54mm_Vertical, symbol Connector_Generic:Conn_01x04
- added J15: EAR, Connector_PinHeader_2.54mm:PinHeader_1x04_P2.54mm_Vertical, symbol Connector_Generic:Conn_01x04
- J1: value Front panel harness 1 -> SWITCHES; footprint Connector_Molex:Molex_KK-396_A-41791-0015_1x15_P3.96mm_Vertical -> Connector_PinHeader_2.54mm:PinHeader_1x19_P2.54mm_Vertical; symbol Connector_Generic:Conn_01x15 -> Connector_Generic:Conn_01x19
- J2: value Front panel harness 2 -> LEDS; footprint Connector_Molex:Molex_KK-396_A-41791-0012_1x12_P3.96mm_Vertical -> Connector_PinHeader_2.54mm:PinHeader_1x05_P2.54mm_Vertical; symbol Connector_Generic:Conn_01x12 -> Connector_Generic:Conn_01x05
Connections:
- net +5V: now also J1.1 (Pin_1), J2.1 (Pin_1); no longer J1.2 (Pin_2)
- net AUDIO_IN: now also J1.17 (Pin_17); no longer J2.8 (Pin_8)
- net AUDIO_OUT: now also J1.10 (Pin_10); no longer J2.7 (Pin_7)
- net CARRIER_EN_N: now also J1.3 (Pin_3); no longer J2.9 (Pin_9)
- net EAR_A: now also J1.18 (Pin_18), J15.1 (Pin_1)
- net EAR_B: now also J1.19 (Pin_19), J15.3 (Pin_3)
- net GND: now also J1.2 (Pin_2), J14.2 (Pin_2), J14.4 (Pin_4), J15.2 (Pin_2), J15.4 (Pin_4); no longer J1.4 (Pin_4), J2.10 (Pin_10)
- net LED_READ_DATA: now also J2.5 (Pin_5); no longer J1.3 (Pin_3)
- net LED_READ_RDY: now also J2.3 (Pin_3); no longer J2.5 (Pin_5)
- net LED_REC_DATA: now also J2.4 (Pin_4); no longer J1.6 (Pin_6)
- net LED_REC_RDY: now also J2.2 (Pin_2); no longer J2.6 (Pin_6)
- net LOCAL_REMOTE: now also J1.9 (Pin_9); no longer J1.8 (Pin_8)
- net MAN_MOTOR: now also J1.4 (Pin_4); no longer J1.11 (Pin_11)
- net MIC_A: now also J1.11 (Pin_11), J14.1 (Pin_1)
- net MIC_B: now also J1.12 (Pin_12), J14.3 (Pin_3)
- net MOTOR_1A: now also J13.1 (Pin_1); no longer J1.1 (Pin_1)
- net MOTOR_1B: now also J13.2 (Pin_2); no longer J1.7 (Pin_7)
- net MOTOR_2A: now also J13.3 (Pin_3); no longer J1.14 (Pin_14)
- net MOTOR_2B: now also J13.4 (Pin_4); no longer J2.1 (Pin_1)
- net READ_RLY_DRV: now also J1.16 (Pin_16); no longer J1.12 (Pin_12)
- net READ_RST: now also J1.8 (Pin_8); no longer J1.9 (Pin_9)
- net READ_SET: now also J1.7 (Pin_7); no longer J2.2 (Pin_2)
- net REC_RLY_DRV: now also J1.13 (Pin_13); no longer J1.10 (Pin_10)
- net REC_RST: now also J1.6 (Pin_6); no longer J2.4 (Pin_4)
- net REC_SET: now also J1.5 (Pin_5); no longer J2.3 (Pin_3)
- net RELAY_1: now also J1.14 (Pin_14); no longer J1.5 (Pin_5)
- net RELAY_2: now also J1.15 (Pin_15); no longer J1.13 (Pin_13)
- no-connect marks 34 -> 31
Other:
- note added: "Front panel jumper pads"
- moved on the sheet: C12, C13, C14, C15, C16, C17, C18, C19, C20, D10, D11, D18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

Commit message: Wired, human-readable schematics with PDF and PNG images
gen.py now lays out each functional group on its own and draws its nets
as real wires (new tools/schroute.py: orthogonal grid router that never
ends, bends or overlaps on another net's wire); every routed net keeps
one label with its name, labels join nets between blocks and sheets, and
unroutable connections fall back to label pairs (17). The front-panel
jumper pads share the front-panel block. Custom 1488/1489 output pins
moved onto the 2.54 mm grid.

build.sh exports schematic/<project>.pdf and, via tools/schimg.py, PNGs
of every sheet and functional block for both boards.

Connectivity unchanged (pin-to-net maps identical for both variants);
ERC 0; both PCBs DRC/parity clean and unchanged. Docs updated.

Co-Authored-By: Claude Opus 5.5 <noreply@anthropic.com>
Other:
- note added: "Generated from docs/ac30_schematica.jpg (SWTPC AC-30 Cassette Tape Switching Schematic), docs/AC30-BOM.md and docs/ac30_wiring1a.jpg. Each block is wired; net labels join the blocks and sheets (identical labels are connected). Transcription notes / assumptions: - Drawing pin-number slips corrected to the real pinouts: IC7D drawn 8->9 (4049: 9->10); IC13C drawn inputs 7,8 (4070: 8,9). - 4053 INH (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"
- note removed: "Front panel jumper pads"
- note removed: "Generated from docs/ac30_schematica.jpg (SWTPC AC-30 Cassette Tape Switching Schematic), docs/AC30-BOM.md and docs/ac30_wiring1a.jpg. Connectivity is by net label: identical labels are connected. Transcription notes / assumptions: - Drawing pin-number slips corrected to the real pinouts: IC7D drawn 8->9 (4049: 9->10); IC13C drawn inputs 7,8 (4070: 8,9). - 4053 INH (pin 6) and VEE (pin 7) are not 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"
- moved on the sheet: C12, C13, C14, C15, C16, C17, C18, C19, C20, D10, D11, D18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
