File: kicad-smt/AC30_SMT_moddemod_power.kicad_sch (KiCad schematic)
At the start: 54 parts, among them IC1 4013, IC2 4001, IC3 4070, IC4 4558, IC5 4013, J12 Power input, Q1 MMBT5088, Q2 MMBT5088, Q3 MMBT5087, Q4 MMBT5088

Commit message: Wired, human-readable schematics with PDF and PNG images
gen.py now lays out each functional group on its own and draws its nets
as real wires (new tools/schroute.py: orthogonal grid router that never
ends, bends or overlaps on another net's wire); every routed net keeps
one label with its name, labels join nets between blocks and sheets, and
unroutable connections fall back to label pairs (17). The front-panel
jumper pads share the front-panel block. Custom 1488/1489 output pins
moved onto the 2.54 mm grid.

build.sh exports schematic/<project>.pdf and, via tools/schimg.py, PNGs
of every sheet and functional block for both boards.

Connectivity unchanged (pin-to-net maps identical for both variants);
ERC 0; both PCBs DRC/parity clean and unchanged. Docs updated.

Co-Authored-By: Claude Opus 5.5 <noreply@anthropic.com>
Other:
- note added: "Generated from docs/ac30_mod_demod.pdf (SWTPC AC-30 Cassette Tape Modulator/Demodulator Schematic). Each block is wired; net labels join the blocks and sheets (identical labels are connected). Transcription notes / assumptions: - IC4 (4558) supply pins are not drawn. The assembly manual says IC4 runs from the +/-7.5 V zener rails (D12/D13 on the power supply sheet). - R16's far end has a terminal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"
- note removed: "Generated from docs/ac30_mod_demod.pdf (SWTPC AC-30 Cassette Tape Modulator/Demodulator Schematic). Connectivity is by net label: identical labels are connected. Transcription notes / assumptions: - IC4 (4558) supply pins are not drawn. The assembly manual says IC4 runs from the +/-7.5 V zener rails (D12/D13 on the power supply sheet). - R16's far end has a terminal dot with no label; taken as +5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"
- moved on the sheet: C1, C10, C11, C2, C23, C24, C25, C3, C4, C5, C6, C7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
